File: hardware/afe-shield/afe-shield.kicad_pcb (KiCad board)
At the start: 2 copper layers, 101.6 x 53.3 mm, 13 parts, among them J1 Power, J2 PWM, J3 Analog, J4 PWM, J5 Analog, J6 Communication, J7 Digital

Commit message: hardware: validate AFE baseline and standardize on KiCad 10
Correct Due header assignments and schematic annotations, integrate original vendor models and offline official references, and add reproducible connectivity and simulation checks.

Document unresolved Stage A performance and PCB release gates, record the proposed PCB development plan, and require KiCad 10.x across benches. Preserve the existing KiCad 10 project migration.
Connections:
- net /*44 renamed /44
- net /*45 renamed /45
- net /*46 renamed /46
- net /*52 renamed /52
- net /A12 renamed /DAC0
- net /A13 renamed /DAC1
- net /A14 renamed /CANRX0
- net /A15 renamed /CANTX0
- net VCC renamed /Vin
- J2 pad 1: /SCL/21 -> /SCL1
- J2 pad 2: /SDA/20 -> /SDA1
Changed lines of the file:
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@@
 	(paper "A4")
 	(title_block
-		(date "mar. 31 mars 2015")
+		(title "Due AFE shield - mechanical template only")
+		(rev "A-design")
+		(comment 1 "Stage A parts not placed or routed. NOT FOR FABRICATION.")
 	)
 	(layers
@@
 	(net 0 "")
 	(net 1 "GND")
-	(net 2 "/*52")
+	(net 2 "/52")
 	(net 3 "/53")
 	(net 4 "/50")
@@
 	(net 6 "/48")
 	(net 7 "/49")
-	(net 8 "/*46")
+	(net 8 "/46")
 	(net 9 "/47")
-	(net 10 "/*44")
-	(net 11 "/*45")
+	(net 10 "/44")
+	(net 11 "/45")
 	(net 12 "/42")
 	(net 13 "/43")
@@
 	(net 46 "/A10")
 	(net 47 "/A11")
-	(net 48 "/A12")
-	(net 49 "/A13")
-	(net 50 "/A14")
-	(net 51 "/A15")
+	(net 48 "/DAC0")
+	(net 49 "/DAC1")
+	(net 50 "/CANRX0")
+	(net 51 "/CANTX0")
 	(net 52 "/AREF")
 	(net 53 "/*13")
@@
 	(net 74 "/SDA{slash}20")
 	(net 75 "/SCL{slash}21")
-	(net 76 "VCC")
+	(net 79 "/SDA1")
+	(net 80 "/SCL1")
+	(net 76 "/Vin")
 	(net 77 "/~{RESET}")
 	(net 78 "unconnected-(J1-Pin_1-Pad1)")
@@
 		)
 		(fp_line
-			(start -3.87 44.51)
+			(start -3.30 44.51)
 			(end 1.33 44.51)
 			(stroke
@@
 				(type solid)
 			)
+			(layer "F.SilkS")
+		)
+		(fp_line
+			(start -3.87 44.0)
+			(end -3.30 44.51)
+			(stroke (width 0.12) (type solid))
 			(layer "F.SilkS")
 		)
@@
 		(fp_line
 			(start -3.87 -1.33)
-			(end -3.87 44.51)
+			(end -3.87 44.0)
 			(stroke
 				(width 0.12)
@@
 			)
 			(remove_unused_layers no)
-			(net 2 "/*52")
+			(net 2 "/52")
 			(pinfunction "Pin_3")
 			(pintype "passive")
@@
 			)
 			(remove_unused_layers no)
-			(net 8 "/*46")
+			(net 8 "/46")
 			(pinfunction "Pin_9")
 			(pintype "passive")
@@
 			)
 			(remove_unused_layers no)
-			(net 10 "/*44")
+			(net 10 "/44")
 			(pinfunction "Pin_11")
 			(pintype "passive")
@@
 			)
 			(remove_unused_layers no)
-			(net 11 "/*45")
+			(net 11 "/45")
 			(pinfunction "Pin_12")
 			(pintype "passive")
@@
 			)
 			(remove_unused_layers no)
-			(net 76 "VCC")
+			(net 76 "/Vin")
 			(pinfunction "Pin_8")
 			(pintype "passive")
@@
 			)
 			(remove_unused_layers no)
-			(net 48 "/A12")
+			(net 48 "/DAC0")
 			(pinfunction "Pin_5")
 			(pintype "passive")
@@
 			)
 			(remove_unused_layers no)
-			(net 49 "/A13")
+			(net 49 "/DAC1")
 			(pinfunction "Pin_6")
 			(pintype "passive")
@@
 			)
 			(remove_unused_layers no)
-			(net 50 "/A14")
+			(net 50 "/CANRX0")
 			(pinfunction "Pin_7")
 			(pintype "passive")
@@
 			)
 			(remove_unused_layers no)
-			(net 51 "/A15")
+			(net 51 "/CANTX0")
 			(pinfunction "Pin_8")
 			(pintype "passive")
@@
 			)
 			(remove_unused_layers no)
-			(net 75 "/SCL{slash}21")
+			(net 80 "/SCL1")
 			(pinfunction "Pin_1")
 			(pintype "passive")
@@
 			)
 			(remove_unused_layers no)
-			(net 74 "/SDA{slash}20")
+			(net 79 "/SDA1")
 			(pinfunction "Pin_2")
 			(pintype "passive")
