File: hardware/afe-shield/afe-shield.kicad_sch (KiCad schematic)
At the start: 7 parts, among them J1 Power, J2 PWM, J3 Analog, J4 PWM, J5 Analog, J6 Communication, J7 Digital

Commit message: hardware: validate AFE baseline and standardize on KiCad 10
Correct Due header assignments and schematic annotations, integrate original vendor models and offline official references, and add reproducible connectivity and simulation checks.

Document unresolved Stage A performance and PCB release gates, record the proposed PCB development plan, and require KiCad 10.x across benches. Preserve the existing KiCad 10 project migration.
Connections:
- net SCL/21: no longer J2.1 (Pin_1)
- net SDA/20: no longer J2.2 (Pin_2)
- net *44 renamed 44
- net *45 renamed 45
- net *46 renamed 46
- net *52 renamed 52
- net A12 renamed DAC0
- net A13 renamed DAC1
- net A14 renamed CANRX0
- net A15 renamed CANTX0
- net VCC renamed Vin
- new net SCL1: J2.1 (Pin_1)
- new net SDA1: J2.2 (Pin_2)
Other:
- sheet reference ports: added none; removed VREF3V0
- note added: "* marks Arduino analogWrite PWM (D2-D13)"
- note added: ".include "sim/sources.cir""
- note added: "Simulation-only Due sources and loads; not PCB parts. Use PSpice compatibility."
- note added: "Stage A: reference and DAC-to-ADC loopback. J5 pins 5-8: DAC0, DAC1, CANRX0, CANTX0 (Due pin names)."
- note removed: "* Indicates a PWM-capable pin"
- note removed: "AFE shield, Stage A. On the Due the positions this template labels A12..A15 are DAC0, DAC1, CANRX0, CANTX0."
Changed lines of the file:
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@@
 		(title "AFE shield for the Arduino Due")
 		(rev "A")
-		(comment 1 "Root: KiCad's Arduino_Mega template; the Due's headers are the Mega's")
+		(comment 1 "Mega-format mechanics; Due-specific signal assignments")
 	)
-	(text "* Indicates a PWM-capable pin"
+	(text "* marks Arduino analogWrite PWM (D2-D13)"
 		(exclude_from_sim no)
 		(at 177.8 180.34 0)
@@
 		)
 	)
-	(label "A15"
+	(label "CANTX0"
 		(at 21.59 102.87 0)
 		(effects
@@
 		)
 	)
-	(label "*44"
+	(label "44"
 		(at 39.37 109.22 270)
 		(effects
@@
 		)
 	)
-	(label "*52"
+	(label "52"
 		(at 29.21 109.22 270)
 		(effects
@@
 		)
 	)
-	(label "A13"
+	(label "DAC1"
 		(at 21.59 97.79 0)
 		(effects
@@
 		)
 	)
-	(label "*45"
+	(label "45"
 		(at 39.37 142.24 90)
 		(effects
@@
 		)
 	)
-	(label "SDA{slash}20"
+	(label "SDA1"
 		(at 74.93 29.21 180)
 		(effects
@@
 		)
 	)
-	(label "A14"
+	(label "CANRX0"
 		(at 21.59 100.33 0)
 		(effects
@@
 		)
 	)
-	(label "*46"
+	(label "46"
 		(at 36.83 109.22 270)
 		(effects
@@
 		)
 	)
-	(label "SCL{slash}21"
+	(label "SCL1"
 		(at 74.93 26.67 180)
 		(effects
@@
 		)
 	)
-	(label "A12"
+	(label "DAC0"
 		(at 21.59 95.25 0)
 		(effects
@@
 		(on_board yes)
 		(dnp no)
-		(property "Reference" "#PWR03"
+		(property "Reference" "#PWR003"
 			(at 31.75 30.48 0)
 			(effects
@@
 			(project "afe-shield"
 				(path "/e63e39d7-6ac0-4ffd-8aa3-1841a4541b55"
-					(reference "#PWR03")
+					(reference "#PWR003")
 					(unit 1)
 				)
@@
 		(on_board yes)
 		(dnp no)
-		(property "Reference" "#PWR02"
+		(property "Reference" "#PWR002"
 			(at 29.21 30.48 0)
 			(effects
@@
 			(project "afe-shield"
 				(path "/e63e39d7-6ac0-4ffd-8aa3-1841a4541b55"
-					(reference "#PWR02")
+					(reference "#PWR002")
 					(unit 1)
 				)
@@
 		(on_board yes)
 		(dnp no)
-		(property "Reference" "#PWR04"
+		(property "Reference" "#PWR004"
 			(at 31.75 58.42 0)
 			(effects
@@
 			(project "afe-shield"
 				(path "/e63e39d7-6ac0-4ffd-8aa3-1841a4541b55"
-					(reference "#PWR04")
+					(reference "#PWR004")
 					(unit 1)
 				)
@@
 		(on_board yes)
 		(dnp no)
-		(property "Reference" "#PWR05"
+		(property "Reference" "#PWR005"
 			(at 64.77 58.42 0)
 			(effects
@@
 			(project "afe-shield"
 				(path "/e63e39d7-6ac0-4ffd-8aa3-1841a4541b55"
-					(reference "#PWR05")
+					(reference "#PWR005")
 					(unit 1)
 				)
@@
 		(on_board yes)
 		(dnp no)
-		(property "Reference" "#PWR07"
+		(property "Reference" "#PWR007"
 			(at 21.59 146.05 0)
 			(effects
@@
 			(project "afe-shield"
 				(path "/e63e39d7-6ac0-4ffd-8aa3-1841a4541b55"
-					(reference "#PWR07")
+					(reference "#PWR007")
 					(unit 1)
 				)
@@
 		(on_board yes)
 		(dnp no)
-		(property "Reference" "#PWR06"
+		(property "Reference" "#PWR006"
 			(at 74.93 115.57 0)
 			(effects
@@
 			(project "afe-shield"
 				(path "/e63e39d7-6ac0-4ffd-8aa3-1841a4541b55"
-					(reference "#PWR06")
-					(unit 1)
-				)
-			)
-		)
-	)
-	(symbol
-		(lib_id "power:VCC")
-		(at 26.67 26.67 0)
-		(unit 1)
-		(exclude_from_sim no)
-		(in_bom yes)
-		(on_board yes)
-		(dnp no)
-		(property "Reference" "#PWR01"
-			(at 26.67 30.48 0)
-			(effects
-				(font
-					(size 1.27 1.27)
-				)
-				(hide yes)
-			)
-		)
-		(property "Value" "VCC"
-			(at 27.051 23.622 90)
-			(effects
-				(font
-					(size 1.27 1.27)
-				)
-				(justify left)
-			)
-		)
-		(property "Footprint" ""
-			(at 26.67 26.67 0)
-			(effects
-				(font
-					(size 1.27 1.27)
-				)
-				(hide yes)
-			)
-		)
-		(property "Datasheet" ""
-			(at 26.67 26.67 0)
-			(effects
-				(font
-					(size 1.27 1.27)
-				)
-				(hide yes)
-			)
-		)
-		(property "Description" "Power symbol creates a global label with name \"VCC\""
-			(at 26.67 26.67 0)
-			(effects
-				(font
-					(size 1.27 1.27)
-				)
-				(hide yes)
-			)
-		)
-		(pin "1"
-		)
-		(instances
-			(project "afe-shield"
-				(path "/e63e39d7-6ac0-4ffd-8aa3-1841a4541b55"
-					(reference "#PWR01")
+					(reference "#PWR006")
 					(unit 1)
 				)
@@
 		)
 		(property "Sheetfile" "reference.kicad_sch"
-			(at 127.0 59.120000000000005 0)
+			(at 127.0 59.12 0)
 			(effects
 				(font
@@
 			)
 		)
-		(pin "VREF3V0" output
-			(at 165.1 48.260000000000005 0)
-			(effects
-				(font
-					(size 1.27 1.27)
-				)
-				(justify right)
-			)
-		)
 		(pin "VREF1V5" output
 			(at 165.1 53.34 0)
@@
 	(wire
 		(pts
-			(xy 165.1 48.260000000000005)
-			(xy 170.18 48.260000000000005)
-		)
-		(stroke
-			(width 0)
-			(type default)
-		)
-	)
-	(label "VREF3V0"
-		(at 170.18 48.260000000000005 0)
-		(effects
-			(font
-				(size 1.27 1.27)
-			)
-			(justify left bottom)
-		)
-	)
-	(wire
-		(pts
 			(xy 165.1 53.34)
 			(xy 170.18 53.34)
@@
 		)
 		(pin "A3" passive
-			(at 165.1 96.52000000000001 0)
+			(at 165.1 96.52 0)
 			(effects
 				(font
@@
 		)
 	)
-	(label "A12"
+	(label "DAC0"
 		(at 121.92 81.28 180)
 		(effects
@@
 		)
 	)
-	(label "A13"
+	(label "DAC1"
 		(at 121.92 86.36 180)
 		(effects
@@
 	(wire
 		(pts
-			(xy 165.1 96.52000000000001)
-			(xy 170.18 96.52000000000001)
+			(xy 165.1 96.52)
+			(xy 170.18 96.52)
 		)
 		(stroke
@@
 	)
 	(label "A3"
-		(at 170.18 96.52000000000001 0)
+		(at 170.18 96.52 0)
 		(effects
 			(font
@@
 		)
 	)
-	(text "AFE shield, Stage A. On the Due the positions this template labels A12..A15 are DAC0, DAC1, CANRX0, CANTX0."
+	(text "Stage A: reference and DAC-to-ADC loopback. J5 pins 5-8: DAC0, DAC1, CANRX0, CANTX0 (Due pin names)."
 		(exclude_from_sim no)
 		(at 127.0 33.02 0)
@@
 	)
 	(embedded_fonts no)
+	(symbol
+		(lib_id "power:PWR_FLAG")
+		(at 85.09 111.76 0)
+		(unit 1)
+		(in_bom no)
+		(on_board yes)
+		(property "Reference" "#FLG03" (at 85.09 115.57 0) (effects (font (size 1.27 1.27)) (hide yes)))
+		(property "Value" "PWR_FLAG" (at 85.09 107.95 0) (effects (font (size 1.27 1.27))))
+		(instances (project "afe-shield" (path "/e63e39d7-6ac0-4ffd-8aa3-1841a4541b55" (reference "#FLG03") (unit 1))))
+	)
+	(wire (pts (xy 74.93 111.76) (xy 85.09 111.76)) (stroke (width 0) (type default)))
+	(text ".include \"sim/sources.cir\""
+		(at 127 157.48 0)
+		(effects (font (size 1.27 1.27)) (justify left bottom))
+	)
+	(text "Simulation-only Due sources and loads; not PCB parts. Use PSpice compatibility."
+		(at 127 162.56 0)
+		(effects (font (size 1.27 1.27)) (justify left bottom))
+	)
 )
