File: hardware/afe-shield/reference.kicad_sch (KiCad schematic)
At the start: 11 parts, among them U1 MCP6024

Commit message: hardware: validate AFE baseline and standardize on KiCad 10
Correct Due header assignments and schematic annotations, integrate original vendor models and offline official references, and add reproducible connectivity and simulation checks.

Document unresolved Stage A performance and PCB release gates, record the proposed PCB development plan, and require KiCad 10.x across benches. Preserve the existing KiCad 10 project migration.
Parts:
- D1: value LM4040DBZ-3.0 -> LM4040-3.0; MPN (none) -> LM4040AIM3-3.0/NOPB
- R3, R4: Tolerance (none) -> 0.1%
- U1: MPN (none) -> MCP6024-E/SL
Other:
- note added: "U1A: verify headroom and stability into the Due AREF ferrite / 100 nF + 100 nF load before closing JP1."
- note removed: "U1A must hold 3.000 V at 250 uA into ADVREF (14 kOhm) on a 3.3 V rail: (check) the headroom with the vendor model."
