File: hardware/afe-shield/pin-driver.kicad_sch (KiCad schematic)
At the start: 16 parts, among them U1 MCP6024

Commit message: hardware: validate AFE baseline and standardize on KiCad 10
Correct Due header assignments and schematic annotations, integrate original vendor models and offline official references, and add reproducible connectivity and simulation checks.

Document unresolved Stage A performance and PCB release gates, record the proposed PCB development plan, and require KiCad 10.x across benches. Preserve the existing KiCad 10 project migration.
Parts:
- C6, R5, R6: Dielectric (none) -> C0G/NP0
- U1: MPN (none) -> MCP6024-E/SL

Commit message: hardware: add AFE acquisition and construction checks
Keep the electrical gate open while making its evidence reproducible.
Separate full-input-step settling from a switched sampling-load screen
fitted to the SAM3X source-impedance relation. Retain the 15-case report,
its input hashes and explicit model limits; do not claim a silicon model
or qualify the hand-wired shield from assumed parasitics.

Correct misplaced capacitor dielectric fields found on R5 and R6,
require 1% driver resistors and 5% C0G capacitors, and validate the
exported BOM. Add strict baseline failure status so completed analyses
cannot silently stand in for passed performance checks.

Preserve official SAM3X and OPA4350 references and the original TI model.
The integrated OPA4350 candidate does not converge, so leave the active
MCP6024 selection unchanged. Document construction and assembly gates.

Validate ERC and BOM checks, eight screening-metric tests, 51 document
reference tests and all 16 reference hashes. An intentional settling
mutation fails its test. The strict baseline exits 2 with four open
findings; PCB template DRC remains unchanged. Preserve vendor whitespace
and original bytes rather than applying project formatting to the model.

Signed-off-by: Jerry Tian <jerryrt@gmail.com>
Parts:
- C5, C7: Dielectric (none) -> C0G/NP0; Tolerance (none) -> 5%
- C6: Tolerance (none) -> 5%
- R5, R6: Dielectric C0G/NP0 -> (none); Tolerance (none) -> 1%
- R7: Tolerance (none) -> 1%
Changed lines of the file:
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@@
 			)
 		)
-		(property "Dielectric" "C0G/NP0" (at 73.66 41.91 0) (effects (font (size 1.27 1.27)) (hide yes)))
+		(property "Tolerance" "1%" (at 66.04 38.1 0) (effects (font (size 1.27 1.27)) (hide yes)))
 	)
 	(wire
@@
 		(pin "2"
 		)
+		(property "Dielectric" "C0G/NP0" (at 73.66 41.91 0) (effects (font (size 1.27 1.27)) (hide yes)))
+		(property "Tolerance" "5%" (at 73.66 41.91 0) (effects (font (size 1.27 1.27)) (hide yes)))
 		(instances
 			(project "afe-shield"
@@
 			)
 		)
-		(property "Dielectric" "C0G/NP0" (at 73.66 62.23 0) (effects (font (size 1.27 1.27)) (hide yes)))
+		(property "Tolerance" "1%" (at 66.04 58.42 0) (effects (font (size 1.27 1.27)) (hide yes)))
 	)
 	(wire
@@
 			)
 		)
-		(property "Dielectric" "C0G/NP0" (at 73.66 82.55 0) (effects (font (size 1.27 1.27)) (hide yes)))
+		(property "Dielectric" "C0G/NP0" (at 73.66 62.23 0) (effects (font (size 1.27 1.27)) (hide yes)))
+		(property "Tolerance" "5%" (at 73.66 62.23 0) (effects (font (size 1.27 1.27)) (hide yes)))
 	)
 	(wire
@@
 		(pin "2"
 		)
+		(property "Tolerance" "1%" (at 66.04 78.74 0) (effects (font (size 1.27 1.27)) (hide yes)))
 		(instances
 			(project "afe-shield"
@@
 		(pin "2"
 		)
+		(property "Dielectric" "C0G/NP0" (at 73.66 82.55 0) (effects (font (size 1.27 1.27)) (hide yes)))
+		(property "Tolerance" "5%" (at 73.66 82.55 0) (effects (font (size 1.27 1.27)) (hide yes)))
 		(instances
 			(project "afe-shield"
